File: SOLoRa.brd (EAGLE design)
At the start: 59.7 x 50.8 mm, 55 parts, among them J1 CONN_USB-MIRCO_10118194, J2 JSTPH, J4 CORTEX_DEBUG_PTH, Q1 RE1C002UNTCL, U1 ATSAMD21G18A-AUT, U2 LIS3DETR, U3 MCP73831T-2ACI/OT, U4 RFM69HCW, U5 LM75, U6 NCP718ASNADJT1G, X1 32.768

Commit message: Version 1.1
Parts:
- removed C14: 1uF, microbuilder:0603-NO
- removed JP7: (no value), microbuilder:1X12_ROUND
- added C11: 22pF, microbuilder:0603-NO
- added J10, J11: (no value), SparkFun-Connectors:1X04_1MM_RA
- added J6: CORTEX_DEBUG_PTH, SparkFun-Connectors:2X5-PTH-1.27MM
- added J7: (no value), microbuilder:1X16_ROUND
- added TP-GND: SE14, solpad:SE14
- C1: value 1uF -> 10µF; device microbuilder:0603-NO -> microbuilder:0805-NO
- C10: value 10uF -> 22pF; device microbuilder:0805-NO -> microbuilder:0603-NO
- C2, C4: value 22pF -> 10µF; device microbuilder:0603-NO -> microbuilder:0805-NO
- C3, C8: value 10µF -> 10uF
- C5, C9: value 10uF -> 1uF; device microbuilder:0805-NO -> microbuilder:0603-NO
- C6: value 10µF -> 1uF; device microbuilder:0805-NO -> microbuilder:0603-NO
- C7: value 1uF -> 10uF; device microbuilder:0603-NO -> microbuilder:0805-NO
- D1, D2: value CUS520,H3F -> BAT54-7-F; device SamacSys_Parts:SOD2513X135N -> _Joes:SOT-23
- J2: value JSTPH -> (none); device microbuilder:JSTPH2 -> microbuilder:1X12_ROUND
- J4: value CORTEX_DEBUG_PTH -> JSTPH; device SparkFun-Connectors:2X5-PTH-1.27MM -> microbuilder:JSTPH2
- JP1: value (none) -> JUMPER-SMT_2_NC_TRACE_NO-SILK; device microbuilder:1X16_ROUND -> SparkFun-Jumpers:SMT-JUMPER_2_NC_TRACE_NO-SILK
- R2: value 1K -> 220K; device microbuilder:0603-NO -> rcl:R0603
- R3: value 220k -> 383K; device microbuilder:0603-NO -> rcl:R0603
- R4: value 383K -> 1K; device rcl:R0603 -> microbuilder:0603-NO
- R5: value 133K -> 22k; device rcl:R0603 -> microbuilder:0603-NO
- R6: value 100K -> 200K; device microbuilder:0603-NO -> rcl:R0603
- R8: value 22k -> 470k
- R9: value 220K -> 100K; device rcl:R0603 -> microbuilder:0603-NO
- U1: value ATSAMD21G18A-AUT -> LM75; device _Joes:QFP50P900X900X120-48N -> _Joes:SO8
- U2: value LIS3DETR -> NCP718ASNADJT1G; device LIS3DETR:LGA16R50P5X3_300X300X100N -> SamacSys_Parts:SOT95P280X100-5N
- U3: value MCP73831T-2ACI/OT -> LIS3DETR; device microbuilder:SOT23-5 -> LIS3DETR:LGA16R50P5X3_300X300X100N
- U4: value RFM69HCW -> MCP73831T-2ACI/OT; device microbuilder:RFMHCW_SMT -> microbuilder:SOT23-5
- U5: value LM75 -> ATSAMD21G18A-AUT; device _Joes:SO8 -> _Joes:QFP50P900X900X120-48N
- U6: value NCP718ASNADJT1G -> RFM69HCW; device SamacSys_Parts:SOT95P280X100-5N -> microbuilder:RFMHCW_SMT
- moved H1 64.0 mm to (5.08, 45.4)
- moved H4 50.0 mm to (55.1, 5.35)
- moved U2 46.1 mm to (9.43, 30.7)
- moved U3 45.6 mm to (55.6, 30.2)
- moved C10 43.5 mm to (19.3, 9.40), turned to 180 degrees
- moved C3 40.6 mm to (55.6, 33.3)
- moved H3 40.0 mm to (5.08, 5.35)
- moved C9 39.9 mm to (16.2, 10.2), turned to 90 degrees
- moved C8 39.8 mm to (55.4, 18.1)
- moved U6 37.1 mm to (44.2, 17.8)
- moved JP1 36.9 mm to (11.2, 39.1), flipped to the bottom, turned to 270 degrees
- moved U1 36.5 mm to (55.6, 38.4), turned to 0 degrees
- moved U5 36.5 mm to (26.7, 16.1), turned to 90 degrees
- moved J2 34.4 mm to (35.6, 30.5), turned to 0 degrees
- moved U4 33.8 mm to (10.7, 22.5)
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- renumbered JP2 to J3, JP4 to J8, JP6 to J9, U$31 to $$U$2, U$32 to $$U$3, U$34 to $$U$1, U$35 to $$U$4
Connections:
- removed net D9: J3.8, R3.2, R6.1, U1.12
- removed net DIO1: JP1.1, U4.7P
- new net D9_A7: J3.8, R8.2, R9.1, U5.12
- new net DIO2: J7.1, U6.8P
- new net PLUS: B1.PLUS, JP1.1
- net !RESET: now also J6.10, J7.16, U5.40; no longer J4.10, JP1.16, U1.40
- net A0: now also J7.12, U5.3; no longer JP1.12, U1.3
- net A1: now also J7.11, U5.7; no longer JP1.11, U1.7
- net A2: now also J7.10, U5.8; no longer JP1.10, U1.8
- net A3: now also J7.9, U5.9; no longer JP1.9, U1.9
- net A4: now also J7.8, U5.10; no longer JP1.8, U1.10
- net A5: now also J7.7, U5.47; no longer JP1.7, U1.47
- net ADJ1: now also R3.1; no longer R4.1
- net ANT: now also U6.1P; no longer U4.1P
- net AREF: now also C9.1, J7.14, U5.4; no longer C14.1, JP1.14, U1.4
- net CHGLED: now also R4.1; no longer R2.1
- net D+: now also U5.34; no longer U1.34
- net D-: now also U5.33; no longer U1.33
- net D0: now also J7.3, U5.16; no longer JP1.3, U1.16
- net D1: now also J7.2, U5.15; no longer JP1.2, U1.15
- net D10: now also U5.27; no longer U1.27
- net D11: now also U5.25, U6.7P; no longer U1.25
- net D12: now also U5.28; no longer U1.28
- net D13: now also U5.26; no longer U1.26
- net D2: now also U5.23; no longer U1.23
- net D3_IRQ: now also U5.14, U6.6P; no longer U1.14, U4.6P
- net D4_RST: now also U5.13, U6.14P; no longer U1.13, U4.14P
- net D5: now also U5.24; no longer U1.24
- net D6: now also U3.11, U5.29; no longer U1.29, U2.11
- net D7: now also U5.30; no longer U1.30
- net D8_CS: now also U5.11, U6.13P; no longer U1.11, U4.13P
- net EN: now also U2.3; no longer U6.3
- net GND: now also C11.2, J10.1, J11.1, J4.1, J6.3, J6.5, J6.9, J7.13, R2.1, R5.2, R6.1, R9.2, TP-GND.MP, U1.4, U1.6, U1.7, U2.2, U3.10, U3.12, U3.5, U3.7, U4.2, U5.18, U5.35, U5.42, U6.16P, U6.2P, U6.9P; no longer C14.2, J2.1, J4.3, J4.5, J4.9, JP1.13, R5.1, R6.2, R8.2, R9.1, U1.18, U1.35, U1.42, U2.10, U2.12, U2.5, U2.7, U3.2, U4.16P, U4.2P, U4.9P, U5.4, U5.6, U5.7, U6.2
- net MISO: now also J7.4, U5.21, U6.10P; no longer JP1.4, U1.21, U4.10P
- net MOSI: now also J7.5, U5.19, U6.11P; no longer JP1.5, U1.19, U4.11P
- net PROG: now also R5.1, U4.5; no longer R8.1, U3.5
- net REGADJ: now also R6.2, U2.4; no longer R5.2, U6.4
- net REGOUT: now also D1.1, R2.2, U2.5; no longer D2.2, R9.2, U6.5
- net SCK: now also J7.6, U5.20, U6.12P; no longer JP1.6, U1.20, U4.12P
- net SCL: now also J10.4, J11.4, U1.2, U3.4, U5.32; no longer U1.32, U2.4, U5.2
- net SDA: now also J10.3, J11.3, U1.1, U3.6, U5.31; no longer U1.31, U2.6, U5.1
- net STAT: now also R4.2, U4.1; no longer R2.2, U3.1
- net SWCLK: now also J6.4, U5.45; no longer J4.4, U1.45
- net SWDIO: now also J6.2, U5.46; no longer J4.2, U1.46
- net VBUS: now also C1.1, D2.3, U2.1, U4.4; no longer C6.1, D1.1, U3.4, U6.1
- net VDD: now also C2.1, C3.1, D1.3, J10.2, J11.2, J6.1, J7.15, JP1.2, R3.2, U1.8, U3.1, U3.14, U3.8, U5.17, U5.36, U5.44, U5.6, U6.5P; no longer B1.PLUS, C10.1, C9.1, D2.1, J4.1, JP1.15, R4.2, U1.17, U1.36, U1.44, U1.6, U2.1, U2.14, U2.8, U4.5P, U5.8
- net VDDCORE: now also C6.1, U5.43; no longer C1.1, U1.43
- net V_BATT: now also C4.1, D2.1, J4.2, R8.1, U4.3; no longer C3.1, D1.2, J2.2, R3.1, U3.3
- net XT1: now also C11.1, U5.1; no longer C2.1, U1.1
- net XT2: now also C10.1, U5.2; no longer C4.1, U1.2
Routing:
- net D9_A7: track 0.00 -> 35.6 mm, vias 0 -> 2
- net D9: track 35.6 -> 0.00 mm, vias 2 -> 0
- net D11: track 14.3 -> 38.3 mm, vias 1 -> 3
- net DIO2: track 0.00 -> 21.1 mm, vias 0 -> 1
- net DIO1: track 18.1 -> 0.00 mm, vias 1 -> 0
- net SCL: track 55.9 -> 67.0 mm
- net SDA: track 56.6 -> 66.9 mm
- net GND: track 0.00 -> 10.0 mm
- net V_BATT: track 30.9 -> 40.4 mm, vias 0 -> 1
- net VDD: track 191.4 -> 194.3 mm, vias 8 -> 10
- net VBUS: track 60.6 -> 62.9 mm
- net PLUS: track 0.00 -> 1.96 mm
- net REGOUT: track 10.00 -> 9.31 mm
Other:
- board text added: "<-QWIIC->"
- board text added: "Accel 6-INT"
- board text added: "Power"
- board text added: "Radio uses: MISO/MOSI/SCK 4-RST,3-IRQ,8-CS"
- board text added: "Rev 1.1"
- board text added: "io2"
- board text removed: "Accel uses: I2C, 6 INT. Temp uses I2C"
- board text removed: "Power Source"
- board text removed: "Radio uses: MISO/MOSI/SCK 4 RST,3 IRQ,8 CS"
- board text removed: "Rev 1.0"
- board text removed: "io1"
