File: SOLoRa.sch (EAGLE design)
At the start: 55 parts, among them J1 CONN_USB-MIRCO_10118194, J2 JSTPH, J4 CORTEX_DEBUG_PTH, Q1 RE1C002UNTCL, U1 ATSAMD21G18A-AUT, U2 LIS3DETR, U3 MCP73831T-2ACI/OT, U4 RFM69HCW, U5 LM75, U6 NCP718ASNADJT1G, X1 32.768

Commit message: Version 1.1
Parts:
- removed C14: 1uF, microbuilder:CAP_CERAMIC0603_NO
- removed JP2, JP4, JP6, JP7: (no value), microbuilder:HEADER-1X12
- added C11: 22pF, microbuilder:CAP_CERAMIC0603_NO
- added J10, J11: (no value), SparkFun-Connectors:QWIIC_CONNECTORJS-1MM
- added J3, J8, J9: (no value), microbuilder:HEADER-1X12
- added J6: CORTEX_DEBUG_PTH, SparkFun-Connectors:CORTEX_DEBUG_PTH
- added J7: (no value), microbuilder:HEADER-1X16ROUND
- added TP-GND: SE14, solpad:SE14
- C1: value 1uF -> 10µF; device microbuilder:CAP_CERAMIC0603_NO -> microbuilder:CAP_CERAMIC0805-NOOUTLINE
- C10: value 10uF -> 22pF; device microbuilder:CAP_CERAMIC0805-NOOUTLINE -> microbuilder:CAP_CERAMIC0603_NO
- C2, C4: value 22pF -> 10µF; device microbuilder:CAP_CERAMIC0603_NO -> microbuilder:CAP_CERAMIC0805-NOOUTLINE
- C3, C8: value 10µF -> 10uF
- C5, C9: value 10uF -> 1uF; device microbuilder:CAP_CERAMIC0805-NOOUTLINE -> microbuilder:CAP_CERAMIC0603_NO
- C6: value 10µF -> 1uF; device microbuilder:CAP_CERAMIC0805-NOOUTLINE -> microbuilder:CAP_CERAMIC0603_NO
- C7: value 1uF -> 10uF; device microbuilder:CAP_CERAMIC0603_NO -> microbuilder:CAP_CERAMIC0805-NOOUTLINE
- D1, D2: value CUS520,H3F -> BAT54-7-F; device SamacSys_Parts:CUS520,H3F -> _Joes:BAT54-7-F
- J2: value JSTPH -> (none); device microbuilder:CON_JST_PH_2PIN -> microbuilder:HEADER-1X12
- J4: value CORTEX_DEBUG_PTH -> JSTPH; device SparkFun-Connectors:CORTEX_DEBUG_PTH -> microbuilder:CON_JST_PH_2PIN
- JP1: value (none) -> JUMPER-SMT_2_NC_TRACE_NO-SILK; device microbuilder:HEADER-1X16ROUND -> SparkFun-Jumpers:JUMPER-SMT_2_NC_TRACE_NO-SILK
- R2: value 1K -> 220K; device microbuilder:RESISTOR_0603_NOOUT -> rcl:R-US_R0603
- R3: value 220k -> 383K; device microbuilder:RESISTOR_0603_NOOUT -> rcl:R-US_R0603
- R4: value 383K -> 1K; device rcl:R-US_R0603 -> microbuilder:RESISTOR_0603_NOOUT
- R5: value 133K -> 22k; device rcl:R-US_R0603 -> microbuilder:RESISTOR_0603_NOOUT
- R6: value 100K -> 200K; device microbuilder:RESISTOR_0603_NOOUT -> rcl:R-US_R0603
- R8: value 22k -> 470k
- R9: value 220K -> 100K; device rcl:R-US_R0603 -> microbuilder:RESISTOR_0603_NOOUT
- U1: value ATSAMD21G18A-AUT -> LM75; device _Joes:ATSAMD21G18A-AUT -> _Joes:LM75
- U2: value LIS3DETR -> NCP718ASNADJT1G; device LIS3DETR:LIS3DETR -> SamacSys_Parts:NCP718ASNADJT1G
- U3: value MCP73831T-2ACI/OT -> LIS3DETR; device microbuilder:MCP73831/2 -> LIS3DETR:LIS3DETR
- U4: value RFM69HCW -> MCP73831T-2ACI/OT; device microbuilder:RFM69HCW_SMT -> microbuilder:MCP73831/2
- U5: value LM75 -> ATSAMD21G18A-AUT; device _Joes:LM75 -> _Joes:ATSAMD21G18A-AUT
- U6: value NCP718ASNADJT1G -> RFM69HCW; device SamacSys_Parts:NCP718ASNADJT1G -> microbuilder:RFM69HCW_SMT
- renumbered U$31 to $$U$2, U$32 to $$U$3, U$34 to $$U$1, U$35 to $$U$4
Connections:
- removed net D9: JP2.8, R3.2, R6.1, U1.PA07
- removed net DIO1: JP1.1, U4.DIO1
- new net D9_A7: J3.8, R8.2, R9.1, U5.PA07
- new net DIO2: J7.1, U6.DIO2
- new net PLUS: B1.PLUS, JP1.1
- net !RESET: now also J6.!RESET, J7.16, U5.!RESETN; no longer J4.!RESET, JP1.16, U1.!RESETN
- net A0: now also J7.12, U5.PA02; no longer JP1.12, U1.PA02
- net A1: now also J7.11, U5.PB08; no longer JP1.11, U1.PB08
- net A2: now also J7.10, U5.PB09; no longer JP1.10, U1.PB09
- net A3: now also J7.9, U5.PA04; no longer JP1.9, U1.PA04
- net A4: now also J7.8, U5.PA05; no longer JP1.8, U1.PA05
- net A5: now also J7.7, U5.PB02; no longer JP1.7, U1.PB02
- net ADJ1: now also R3.1; no longer R4.1
- net ANT: now also U6.ANT; no longer U4.ANT
- net AREF: now also C9.1, J7.14, U5.PA03; no longer C14.1, JP1.14, U1.PA03
- net CHGLED: now also R4.1; no longer R2.1
- net D+: now also U5.PA25; no longer U1.PA25
- net D-: now also U5.PA24; no longer U1.PA24
- net D0: now also J7.3, U5.PA11; no longer JP1.3, U1.PA11
- net D1: now also J7.2, U5.PA10; no longer JP1.2, U1.PA10
- net D10: now also J3.7, U5.PA18; no longer JP2.7, U1.PA18
- net D11: now also J3.6, U5.PA16, U6.DIO1; no longer JP2.6, U1.PA16
- net D12: now also J3.5, U5.PA19; no longer JP2.5, U1.PA19
- net D13: now also J3.4, U5.PA17; no longer JP2.4, U1.PA17
- net D2: now also U5.PA14; no longer U1.PA14
- net D3_IRQ: now also U5.PA09, U6.DIO0; no longer U1.PA09, U4.DIO0
- net D4_RST: now also U5.PA08, U6.RESET; no longer U1.PA08, U4.RESET
- net D5: now also J3.10, U5.PA15; no longer JP2.10, U1.PA15
- net D6: now also J3.9, U3.INT1, U5.PA20; no longer JP2.9, U1.PA20, U2.INT1
- net D7: now also U5.PA21; no longer U1.PA21
- net D8_CS: now also U5.PA06, U6.NSS; no longer U1.PA06, U4.NSS
- net EN: now also J3.2, U2.EN; no longer JP2.2, U6.EN
- net GND: now also C11.2, J10.1, J11.1, J4.1, J6.GND@3, J6.GND@5, J6.GNDDTCT, J7.13, J8.1, J8.10, J8.11, J8.12, J8.2, J8.3, J8.4, J8.5, J8.6, J8.7, J8.8, J8.9, R2.1, R5.2, R6.1, R9.2, TP-GND.MP, U1.A0, U1.A1, U1.A2, U1.GND, U3.GND, U3.RES, U3.SDO/SA0, U4.VSS, U5.GND1, U5.GND2, U5.GND3, U5.GNDANA, U6.GND@1, U6.GND@2, U6.GND@3; no longer C14.2, J2.1, J4.GND@3, J4.GND@5, J4.GNDDTCT, JP1.13, JP4.1, JP4.10, JP4.11, JP4.12, JP4.2, JP4.3, JP4.4, JP4.5, JP4.6, JP4.7, JP4.8, JP4.9, R5.1, R6.2, R8.2, R9.1, U1.GND1, U1.GND2, U1.GND3, U1.GNDANA, U2.RES, U2.SDO/SA0, U3.VSS, U4.GND@1, U4.GND@2, U4.GND@3, U5.A0, U5.A1, U5.A2, U5.GND, U6.GND
- net MISO: now also J7.4, U5.PA12, U6.MISO; no longer JP1.4, U1.PA12, U4.MISO
- net MOSI: now also J7.5, U5.PB10, U6.MOSI; no longer JP1.5, U1.PB10, U4.MOSI
- net PROG: now also R5.1, U4.PROG; no longer R8.1, U3.PROG
- net REGADJ: now also R6.2, U2.ADJ; no longer R5.2, U6.ADJ
- net REGOUT: now also D1.EPAD1, R2.2, U2.OUT; no longer D2.A, R9.2, U6.OUT
- net SCK: now also J7.6, U5.PB11, U6.SCK; no longer JP1.6, U1.PB11, U4.SCK
- net SCL: now also J10.4, J11.4, J3.11, U1.SCL, U3.SCL/SPC, U5.PA23; no longer JP2.11, U1.PA23, U2.SCL/SPC, U5.SCL
- net SDA: now also J10.3, J11.3, J3.12, U1.SDA, U3.SDA/SDI/SDO, U5.PA22; no longer JP2.12, U1.PA22, U2.SDA/SDI/SDO, U5.SDA
- net STAT: now also R4.2, U4.STAT; no longer R2.2, U3.STAT
- net SWCLK: now also J6.SWDCLK/TCK, U5.PA30; no longer J4.SWDCLK/TCK, U1.PA30
- net SWDIO: now also J6.SWDIO/TMS, U5.PA31; no longer J4.SWDIO/TMS, U1.PA31
- net VBUS: now also C1.1, D2.EPAD3, J3.3, U2.IN, U4.VDD; no longer C6.1, D1.K, JP2.3, U3.VDD, U6.IN
- net VDD: now also C2.1, C3.1, D1.EPAD3, J10.2, J11.2, J6.VCC, J7.15, J9.1, J9.10, J9.11, J9.12, J9.2, J9.3, J9.4, J9.5, J9.6, J9.7, J9.8, J9.9, JP1.2, R3.2, U1.VCC, U3.CS, U3.VDD, U3.VDD_IO, U5.VDDANA, U5.VDDIN, U5.VDDIO1, U5.VDDIO2, U6.VDD; no longer B1.PLUS, C10.1, C9.1, D2.K, J4.VCC, JP1.15, JP6.1, JP6.10, JP6.11, JP6.12, JP6.2, JP6.3, JP6.4, JP6.5, JP6.6, JP6.7, JP6.8, JP6.9, R4.2, U1.VDDANA, U1.VDDIN, U1.VDDIO1, U1.VDDIO2, U2.CS, U2.VDD, U2.VDD_IO, U4.VDD, U5.VCC
- net VDDCORE: now also C6.1, U5.VDDCORE; no longer C1.1, U1.VDDCORE
- net V_BATT: now also C4.1, D2.EPAD1, J3.1, J4.2, R8.1, U4.VBAT; no longer C3.1, D1.A, J2.2, JP2.1, R3.1, U3.VBAT
- net XT1: now also C11.1, U5.PA00; no longer C2.1, U1.PA00
- net XT2: now also C10.1, U5.PA01; no longer C4.1, U1.PA01
Other:
- note added: "(Cur Meas)"
- note added: "0.88V 0.77V 0.53V"
- note added: "1.00V 0.80V 0.60V"
- note added: "1.1"
- note added: "402K"
- note added: "470K"
- note added: "5V 4V 3V"
- note added: "Feather Wing Compatible"
- note added: "R5 Value VDD (V) 200K 3.55V * 220K 3.3V"
- note added: "RCR123A LiFePo4 Cell *Use B1 with Solar Cell only Also, set VDD to ~3.55V"
- note added: "Use ADC 1V internal reference for battery voltage measurements"
- note added: "V_BATT R3(K-Ohm) D9(V)"
- note added: "header pads"
- note added: "symbols for hole & fiducial features"
- note removed: "1.0"
- note removed: "2A Max Discharge"
- note removed: "80mA Max Charge"
- note removed: "RCR123A LiFePo4 Cell (Use with Solar Cell only)"
- note removed: "~3.55V"
